Commit message: Set no vel/acc limits. Comment out joint_state_publisher. Fixes to caster wheel. nadie.urdf has fixes for plugins.

File: nadie_control/urdf/caster.urdf.xacro (robot description, xacro)
@@ -4,10 +4,10 @@
 		<link name="${wheel_prefix}_wheel_link">
 			<inertial>
-				<mass value="2.637" />
-				<origin rpy="0 0 0" xyz="0 0 0" />
+				<mass value="0.01" />
+				<origin xyz="0 0 0" />
 				<inertia  ixx="0.02467" ixy="0" ixz="0" iyy="0.04411" iyz="0" izz="0.02467" />
 			</inertial>
 			<visual>
-				<origin xyz="0 0 0" rpy="1.5708 0 0" />
+				<origin xyz="0 0 0" rpy="${M_PI/2} 0 0" />
 				<geometry>
 			        <cylinder length="${wheel_width}" radius="${wheel_radius}" />
@@ -16,5 +16,5 @@
 			</visual>
 			<collision>
-				<origin xyz="0 0 0" rpy="1.5708 0 0" />
+				<origin xyz="0 0 0" rpy="${M_PI/2} 0 0" />
 				<geometry>
 			        <cylinder length="${wheel_width}" radius="${wheel_radius}" />
@@ -23,13 +23,10 @@
 		</link>
 		<gazebo reference="${wheel_prefix}_wheel_link">
-			<kp value="10000000.0" />
-			<kd value="1.0" />
-			<fdir1 value="1 0 0"/>
 		</gazebo>
-		<joint name="${wheel_prefix}_wheel" type="continuous">
+		<joint name="${wheel_prefix}_wheel" type="fixed">
 			<parent link="base_link"/>
 			<child link="${wheel_prefix}_wheel_link"/>
 			<xacro:insert_block name="joint_pose"/>
-			<axis xyz="0 1 0" rpy="0 0 0" />
+			<!--axis xyz="0 1 0" rpy="0 0 0" /-->
 		</joint>
 	</xacro:macro>

File: nadie_control/urdf/nadie.xacro (robot description, xacro)
@@ -31,10 +31,11 @@
   <gazebo>
     <plugin name="differential_drive_controller" filename="libgazebo_ros_diff_drive.so">
-      <commandTopic>cmd_vel</commandTopic> <!-- cmd_vel -->
+      <commandTopic>/nadie/diff_drive_controller/cmd_vel</commandTopic> <!-- cmd_vel -->
+      <legacyMode>true</legacyMode> <!-- If using DefaultRobotHWSim, set this to "true" to fix namespace issue -->
       <leftJoint>front_left_wheel</leftJoint> <!-- left_joint -->
       <odometryFrame>odom</odometryFrame> <!-- odom -->
-      <odometryTopic>odom</odometryTopic> <!-- odom -->
+      <odometryTopic>/nadie/diff_drive_controller/odom</odometryTopic> <!-- odom -->
       <odometrySource>world</odometrySource> <!-- world (in {world, encoder} ) -->
-      <publishTf>true</publishTf> <!-- true, if true pub <odometryTopic> -->
+      <publishTf>false</publishTf> <!-- true, if true pub <odometryTopic> -->
       <publishWheelJointState>false</publishWheelJointState> <!-- false, if true pub "joint_states" -->
       <publishWheelTF>false</publishWheelTF> <!-- false -->
@@ -48,8 +49,10 @@
     </plugin>
     <plugin name="gazebo_ros_control" filename="libgazebo_ros_control.so">
-      <robotNamespace>$(arg robot_namespace)</robotNamespace>
-      <robotNamespace>/nadie</robotNamespace>
-      <legacyModeNS>true</legacyModeNS>
-      <robotSimType>gazebo_ros_control/DefaultRobotHWSim</robotSimType>
+      <!-- controlPeriod defaults to parent_model_->GetWorld()->Physics()->GetMaxStepSize() -->
+      <!-- eStopTopic if specified, subscribe to this topic and capture 'data' value -->
+      <legacyModeNS>true</legacyModeNS> <!-- If using DefaultRobotHWSim, set this to "true" to fix namespace issue -->
+      <robotNamespace>$(arg robot_namespace)</robotNamespace> <!-- parent_model_->GetName() -->
+      <robotParam>robot_description</robotParam> <!-- robot_description -->
+      <robotSimType>gazebo_ros_control/DefaultRobotHWSim</robotSimType> <!-- gazebo_ros_control/DefaultRobotHWSim, which becomes the controller manager -->
     </plugin>
   </gazebo>

File: nadie_control/urdf/wheel.urdf.xacro (robot description, xacro)
@@ -6,5 +6,4 @@
 				<mass value="2.637" />
 				<origin xyz="0 0 0" />
-				<cylinder_inertia m="5" r="0.1" h="0.05"/>
 				<inertia  ixx="0.02467" ixy="0" ixz="0" iyy="0.04411" iyz="0" izz="0.02467" />
 			</inertial>
