Commit message: Getting closer. cmd_vel moves forward but no angular movement

File: nadie_control/urdf/nadie.xacro (robot description, xacro)
@@ -30,10 +30,32 @@
   <!--xacro:include filename="$(find m1)/robots/m1.gazebo" /-->
   <gazebo>
-    <plugin name="gazebo_ros_control" filename="libgazebo_ros_control.so">
-      <!--robotNamespace>$(arg robot_namespace)</robotNamespace-->
+    <plugin name="differential_drive_controller" filename="libgazebo_ros_diff_drive.so">
+      <alwaysOn>true</alwaysOn>
+      <commandTopic>cmd_vel</commandTopic>
+      <legacyMode>false</legacyMode>
+      <leftJoint>front_left_wheel</leftJoint>
+      <odometryFrame>odom</odometryFrame>
+      <odometrySource>true</odometrySource>
+      <odometryTopic>odom</odometryTopic>
+      <publishOdomTF>true</publishOdomTF>
+      <publishTf>true</publishTf>
+      <publishWheelJointState>false</publishWheelJointState>
+      <publishWheelTF>true</publishWheelTF>
+      <rightJoint>front_right_wheel</rightJoint>
+      <robotBaseFrame>base_link</robotBaseFrame>
+      <rosDebugLevel>Debug</rosDebugLevel>
+      <torque>20</torque>
+      <updateRate>20</updateRate>
+      <wheelAcceleration>1</wheelAcceleration>
+      <wheelDiameter>${2*wheel_radius}</wheelDiameter>
+      <wheelSeparation>${body_width+(2*wheel_spacer)+wheel_width}</wheelSeparation>
+      <wheelTorque>20</wheelTorque>
+    </plugin>
+    <!--plugin name="gazebo_ros_control" filename="libgazebo_ros_control.so">
+      <!- -robotNamespace>$(arg robot_namespace)</robotNamespace- ->
       <robotNamespace>/nadie</robotNamespace>
       <legacyModeNS>true</legacyModeNS>
-]     <!--robotSimType>gazebo_ros_control/DefaultRobotHWSim</robotSimType-->
-    </plugin>
+      <robotSimType>gazebo_ros_control/DefaultRobotHWSim</robotSimType>
+    </plugin-->
   </gazebo>
   <!--gazebo>

File: nadie_control/urdf/wheel.urdf.xacro (robot description, xacro)
@@ -6,4 +6,5 @@
 				<mass value="2.637" />
 				<origin xyz="0 0 0" />
+				<cylinder_inertia m="5" r="0.1" h="0.05"/>
 				<inertia  ixx="0.02467" ixy="0" ixz="0" iyy="0.04411" iyz="0" izz="0.02467" />
 			</inertial>
@@ -34,4 +35,6 @@
 			<xacro:insert_block name="joint_pose"/>
 			<axis xyz="0 1 0" rpy="0 0 0" />
+		    <limit effort="100" velocity="100"/>
+		    <joint_properties damping="0.0" friction="0.0"/>
 		</joint>
 		<transmission name="${wheel_prefix}_wheel_trans" type="SimpleTransmission">

Commit message: Snapshot on way to having nav stack working

File: nadie_control/urdf/nadie.xacro (robot description, xacro)
@@ -4,5 +4,5 @@
   <xacro:include filename="$(find nadie_control)/urdf/caster.urdf.xacro" />
   <xacro:include filename="$(find nadie_control)/urdf/wheel.urdf.xacro" />
-  <!--xacro:include filename="$(find motor_controller)/urdf/nadie.gazebo" /-->
+  <!--xacro:include filename="$(find nadie_control)/urdf/lidar_sim.xacro" /-->
   <xacro:property name="M_PI" value="3.14159"/>
   <xacro:property name="wheel_vertical_offset" value="0.03282" />
@@ -110,4 +110,65 @@
     <origin xyz="${fwheel_offset} 0 ${wheel_vertical_offset}" rpy="0 0 0" />
   </xacro:caster>
+  <joint name="hokuyo_joint" type="fixed">
+    <axis xyz="0 1 0" />
+    <origin xyz="${lidar_x_offset} 0 ${lidar_z_offset}" rpy="0 0 0"/>
+    <parent link="base_link"/>
+    <child link="hokuyo_link"/>
+  </joint>
+  <!-- Hokuyo Laser -->
+  <link name="hokuyo_link">
+    <collision>
+      <origin xyz="0 0 0" rpy="0 0 0"/>
+      <geometry>
+    <box size="0.1 0.1 0.1"/>
+      </geometry>
+    </collision>
+    <visual>
+      <origin xyz="0 0 0" rpy="0 0 0"/>
+      <geometry>
+        <mesh filename="package://nadie_control/meshes/hokuyo.dae"/>
+      </geometry>
+    </visual>
+    <inertial>
+      <mass value="1e-5" />
+      <origin xyz="0 0 0" rpy="0 0 0"/>
+      <inertia ixx="1e-6" ixy="0" ixz="0" iyy="1e-6" iyz="0" izz="1e-6" />
+    </inertial>
+  </link>
+  <gazebo reference="hokuyo_link">
+    <sensor type="ray" name="head_hokuyo_sensor">
+      <pose>0 0 0 0 0 0</pose>
+      <visualize>true</visualize>
+      <update_rate>7</update_rate>
+      <ray>
+        <scan>
+          <horizontal>
+            <samples>360</samples>
+            <resolution>1</resolution>
+            <min_angle>-3.14159</min_angle>
+            <max_angle>3.14159</max_angle>
+          </horizontal>
+        </scan>
+        <range>
+          <min>0.10</min>
+          <max>6.0</max>
+          <resolution>0.01</resolution>
+        </range>
+        <noise>
+          <type>gaussian</type>
+          <!-- Noise parameters based on published spec for Hokuyo laser
+               achieving "+-30mm" accuracy at range < 10m.  A mean of 0.0m and
+               stddev of 0.01m will put 99.7% of samples within 0.03m of the true
+               reading. -->
+          <mean>0.0</mean>
+          <stddev>0.01</stddev>
+        </noise>
+      </ray>
+      <plugin name="gazebo_ros_head_hokuyo_controller" filename="libgazebo_ros_laser.so">
+        <topicName>/scan</topicName>
+        <frameName>hokuyo_link</frameName>
+      </plugin>
+    </sensor>
+  </gazebo>
   <!--link name="neato">
     <collision>

Commit message: Snapshot, odom is still flaky in sumulation

File: nadie_control/urdf/nadie.xacro (robot description, xacro)
@@ -30,29 +30,11 @@
   <!--xacro:include filename="$(find m1)/robots/m1.gazebo" /-->
   <gazebo>
-    <plugin name="differential_drive_controller" filename="libgazebo_ros_diff_drive.so">
-      <commandTopic>/nadie/diff_drive_controller/cmd_vel</commandTopic> <!-- cmd_vel -->
-      <legacyMode>true</legacyMode> <!-- If using DefaultRobotHWSim, set this to "true" to fix namespace issue -->
-      <leftJoint>front_left_wheel</leftJoint> <!-- left_joint -->
-      <odometryFrame>odom</odometryFrame> <!-- odom -->
-      <odometryTopic>/nadie/diff_drive_controller/odom</odometryTopic> <!-- odom -->
-      <odometrySource>world</odometrySource> <!-- world (in {world, encoder} ) -->
-      <publishTf>false</publishTf> <!-- true, if true pub <odometryTopic> -->
-      <publishWheelJointState>false</publishWheelJointState> <!-- false, if true pub "joint_states" -->
-      <publishWheelTF>false</publishWheelTF> <!-- false -->
-      <rightJoint>front_right_wheel</rightJoint> <!-- right_joint -->
-      <robotBaseFrame>base_link</robotBaseFrame> <!-- base_footprint -->
-      <updateRate>20</updateRate> <!-- 100 -->
-      <wheelAcceleration>1</wheelAcceleration> <!-- 0.0 -->
-      <wheelDiameter>${2*wheel_radius}</wheelDiameter> <!-- 0.15 -->
-      <wheelSeparation>${body_width+(2*wheel_spacer)+wheel_width}</wheelSeparation> <!-- 0.34 -->
-      <wheelTorque>20</wheelTorque> <!-- 5.0 -->
-    </plugin>
     <plugin name="gazebo_ros_control" filename="libgazebo_ros_control.so">
       <!-- controlPeriod defaults to parent_model_->GetWorld()->Physics()->GetMaxStepSize() -->
       <!-- eStopTopic if specified, subscribe to this topic and capture 'data' value -->
-      <legacyModeNS>true</legacyModeNS> <!-- If using DefaultRobotHWSim, set this to "true" to fix namespace issue -->
+      <legacyModeNS>false</legacyModeNS> <!-- If using DefaultRobotHWSim, set this to "true" to fix namespace issue -->
       <robotNamespace>$(arg robot_namespace)</robotNamespace> <!-- parent_model_->GetName() -->
-      <robotParam>robot_description</robotParam> <!-- robot_description -->
-      <robotSimType>gazebo_ros_control/DefaultRobotHWSim</robotSimType> <!-- gazebo_ros_control/DefaultRobotHWSim, which becomes the controller manager -->
+      <!--robotParam>robot_description</robotParam--> <!-- robot_description -->
+      <!--robotSimType>gazebo_ros_control/DefaultRobotHWSim</robotSimType--> <!-- gazebo_ros_control/DefaultRobotHWSim, which becomes the controller manager -->
     </plugin>
   </gazebo>
@@ -110,10 +92,4 @@
     <origin xyz="${fwheel_offset} 0 ${wheel_vertical_offset}" rpy="0 0 0" />
   </xacro:caster>
-  <joint name="hokuyo_joint" type="fixed">
-    <axis xyz="0 1 0" />
-    <origin xyz="${lidar_x_offset} 0 ${lidar_z_offset}" rpy="0 0 0"/>
-    <parent link="base_link"/>
-    <child link="hokuyo_link"/>
-  </joint>
   <!-- Hokuyo Laser -->
   <link name="hokuyo_link">
@@ -121,5 +97,5 @@
       <origin xyz="0 0 0" rpy="0 0 0"/>
       <geometry>
-    <box size="0.1 0.1 0.1"/>
+        <box size="0.1 0.1 0.1"/>
       </geometry>
     </collision>
@@ -136,4 +112,10 @@
     </inertial>
   </link>
+  <joint name="hokuyo_joint" type="fixed">
+    <axis xyz="0 1 0" />
+    <origin xyz="${lidar_x_offset} 0 ${lidar_z_offset}" rpy="0 0 0"/>
+    <parent link="base_link"/>
+    <child link="hokuyo_link"/>
+  </joint>
   <gazebo reference="hokuyo_link">
     <sensor type="ray" name="head_hokuyo_sensor">
@@ -157,8 +139,4 @@
         <noise>
           <type>gaussian</type>
-          <!-- Noise parameters based on published spec for Hokuyo laser
-               achieving "+-30mm" accuracy at range < 10m.  A mean of 0.0m and
-               stddev of 0.01m will put 99.7% of samples within 0.03m of the true
-               reading. -->
           <mean>0.0</mean>
           <stddev>0.01</stddev>
@@ -166,5 +144,5 @@
       </ray>
       <plugin name="gazebo_ros_head_hokuyo_controller" filename="libgazebo_ros_laser.so">
-        <alwaysOn>true</alwaysOn>
+        <alwaysOn>false</alwaysOn>
         <!--robotNamespace></robotNamespace-->
         <topicName>/scan</topicName>
