Commit message: Robot/joint state publishers working, control launcher is not

File: nadie_description/urdf/gazebo.urdf.xacro (robot description, xacro)
@@ -19,14 +19,4 @@
 -->
 <robot xmlns:xacro="http://ros.org/wiki/xacro" name="nadie">
-  <gazebo>
-    <plugin name="gazebo_ros_control" filename="libgazebo_ros_control.so">
-      <!-- controlPeriod defaults to parent_model_->GetWorld()->Physics()->GetMaxStepSize() -->
-      <!-- eStopTopic if specified, subscribe to this topic and capture 'data' value -->
-      <legacyModeNS>false</legacyModeNS> <!-- If using DefaultRobotHWSim, set this to "true" to fix namespace issue -->
-      <robotNamespace>$(arg robot_namespace)</robotNamespace> <!-- parent_model_->GetName() -->
-      <!--robotParam>robot_description</robotParam--> <!-- robot_description -->
-      <!--robotSimType>gazebo_ros_control/DefaultRobotHWSim</robotSimType--> <!-- gazebo_ros_control/DefaultRobotHWSim, which becomes the controller manager -->
-    </plugin>
-  </gazebo>
   <gazebo reference="hokuyo_link">
     <sensor type="ray" name="head_hokuyo_sensor">

File: nadie_description/urdf/nadie.urdf.xacro (robot description, xacro)
@@ -20,5 +20,11 @@
 <robot xmlns:xacro="http://ros.org/wiki/xacro" name="nadie">
   <xacro:arg name="robot_namespace" default="/nadie" />
-  <xacro:include filename="$(find nadie_description)/urdf/caster.urdf.xacro" />
+  <gazebo>
+    <plugin name="gazebo_ros_control" filename="libgazebo_ros_control.so">
+      <legacyModeNS>true</legacyModeNS> <!-- If using DefaultRobotHWSim, set this to "true" to fix namespace issue -->
+      <robotNamespace>$(arg robot_namespace)</robotNamespace> <!-- parent_model_->GetName() -->
+    </plugin>
+  </gazebo>
+ <xacro:include filename="$(find nadie_description)/urdf/caster.urdf.xacro" />
   <xacro:include filename="$(find nadie_description)/urdf/wheel.urdf.xacro" />
   <!--xacro:include filename="$(find nadie_description)/urdf/lidar_sim.xacro" /-->
@@ -99,31 +105,5 @@
     <origin xyz="${fwheel_offset} 0 ${wheel_vertical_offset}" rpy="0 0 0" />
   </xacro:caster>
-  <!-- Hokuyo Laser -->
-  <link name="hokuyo_link">
-    <collision>
-      <origin xyz="0 0 0" rpy="0 0 0"/>
-      <geometry>
-        <box size="0.1 0.1 0.1"/>
-      </geometry>
-    </collision>
-    <visual>
-      <origin xyz="0 0 0" rpy="0 0 0"/>
-      <geometry>
-        <mesh filename="package://nadie_description/meshes/hokuyo.dae"/>
-      </geometry>
-    </visual>
-    <inertial>
-      <mass value="1e-5" />
-      <origin xyz="0 0 0" rpy="0 0 0"/>
-      <inertia ixx="1e-6" ixy="0" ixz="0" iyy="1e-6" iyz="0" izz="1e-6" />
-    </inertial>
-  </link>
-  <joint name="hokuyo_joint" type="fixed">
-    <axis xyz="0 1 0" />
-    <origin xyz="${lidar_x_offset} 0 ${lidar_z_offset}" rpy="0 0 0"/>
-    <parent link="base_link"/>
-    <child link="hokuyo_link"/>
-  </joint>
-  <!--link name="neato">
+  <link name="neato">
     <collision>
       <geometry>
@@ -154,4 +134,4 @@
     <child link="neato"/>
     <origin xyz="${lidar_x_offset} 0  ${lidar_z_offset}" rpy="0 0 0"/>
-  </joint-->
+  </joint>
 </robot>
