Commit message: Separating rviz

File: nadie_description/urdf/caster.urdf.xacro (robot description, xacro)
@@ -1,3 +1,21 @@
 <?xml version="1.0"?>
+<!--
+Copyright (c) 2018 Michael Wimble
+Permission is hereby granted, free of charge, to any person obtaining a copy
+of this software and associated documentation files (the "Software"), to deal
+in the Software without restriction, including without limitation the rights
+to use, copy, modify, merge, publish, distribute, sublicense, and/or sell
+copies of the Software, and to permit persons to whom the Software is
+furnished to do so, subject to the following conditions:
+The above copyright notice and this permission notice shall be included in all
+copies or substantial portions of the Software.
+THE SOFTWARE IS PROVIDED "AS IS", WITHOUT WARRANTY OF ANY KIND, EXPRESS OR
+IMPLIED, INCLUDING BUT NOT LIMITED TO THE WARRANTIES OF MERCHANTABILITY,
+FITNESS FOR A PARTICULAR PURPOSE AND NONINFRINGEMENT. IN NO EVENT SHALL THE
+AUTHORS OR COPYRIGHT HOLDERS BE LIABLE FOR ANY CLAIM, DAMAGES OR OTHER
+LIABILITY, WHETHER IN AN ACTION OF CONTRACT, TORT OR OTHERWISE, ARISING FROM,
+OUT OF OR IN CONNECTION WITH THE SOFTWARE OR THE USE OR OTHER DEALINGS IN THE
+SOFTWARE.
+-->
 <robot xmlns:xacro="http://ros.org/wiki/xacro" name="caster">
 	<xacro:macro name="caster" params="wheel_prefix *joint_pose">

File: nadie_description/urdf/gazebo.urdf.xacro (robot description, xacro)
@@ -18,56 +18,36 @@
 SOFTWARE.
 -->
-<robot xmlns:xacro="http://ros.org/wiki/xacro" name="lidar_sim">
-  <joint name="hokuyo_joint" type="fixed">
-    <axis xyz="0 1 0" />
-    <origin xyz="0 0 0." rpy="${lidar_x_offset} 0 ${lidar_z_offset}"/>
-    <parent link="base_link"/>
-    <child link="hokuyo_link"/>
-  </joint>
-  <!-- Hokuyo Laser -->
-  <link name="hokuyo_link">
-    <collision>
-      <origin xyz="0 0 0" rpy="0 0 0"/>
-      <geometry>
-    <box size="0.1 0.1 0.1"/>
-      </geometry>
-    </collision>
-    <visual>
-      <origin xyz="0 0 0" rpy="0 0 0"/>
-      <geometry>
-        <mesh filename="package://nadie_control/meshes/hokuyo.dae"/>
-      </geometry>
-    </visual>
-    <inertial>
-      <mass value="1e-5" />
-      <origin xyz="0 0 0" rpy="0 0 0"/>
-      <inertia ixx="1e-6" ixy="0" ixz="0" iyy="1e-6" iyz="0" izz="1e-6" />
-    </inertial>
-  </link>
+<robot xmlns:xacro="http://ros.org/wiki/xacro" name="nadie">
+  <gazebo>
+    <plugin name="gazebo_ros_control" filename="libgazebo_ros_control.so">
+      <!-- controlPeriod defaults to parent_model_->GetWorld()->Physics()->GetMaxStepSize() -->
+      <!-- eStopTopic if specified, subscribe to this topic and capture 'data' value -->
+      <legacyModeNS>false</legacyModeNS> <!-- If using DefaultRobotHWSim, set this to "true" to fix namespace issue -->
+      <robotNamespace>$(arg robot_namespace)</robotNamespace> <!-- parent_model_->GetName() -->
+      <!--robotParam>robot_description</robotParam--> <!-- robot_description -->
+      <!--robotSimType>gazebo_ros_control/DefaultRobotHWSim</robotSimType--> <!-- gazebo_ros_control/DefaultRobotHWSim, which becomes the controller manager -->
+    </plugin>
+  </gazebo>
   <gazebo reference="hokuyo_link">
     <sensor type="ray" name="head_hokuyo_sensor">
       <pose>0 0 0 0 0 0</pose>
-      <visualize>false</visualize>
-      <update_rate>40</update_rate>
+      <visualize>true</visualize>
+      <update_rate>7</update_rate>
       <ray>
         <scan>
           <horizontal>
-            <samples>720</samples>
+            <samples>360</samples>
             <resolution>1</resolution>
-            <min_angle>-1.570796</min_angle>
-            <max_angle>1.570796</max_angle>
+            <min_angle>-3.14159</min_angle>
+            <max_angle>3.14159</max_angle>
           </horizontal>
         </scan>
         <range>
           <min>0.10</min>
-          <max>30.0</max>
+          <max>10.0</max>
           <resolution>0.01</resolution>
         </range>
         <noise>
           <type>gaussian</type>
-          <!-- Noise parameters based on published spec for Hokuyo laser
-               achieving "+-30mm" accuracy at range < 10m.  A mean of 0.0m and
-               stddev of 0.01m will put 99.7% of samples within 0.03m of the true
-               reading. -->
           <mean>0.0</mean>
           <stddev>0.01</stddev>
@@ -75,5 +55,8 @@
       </ray>
       <plugin name="gazebo_ros_head_hokuyo_controller" filename="libgazebo_ros_laser.so">
+        <alwaysOn>false</alwaysOn>
+        <!--robotNamespace></robotNamespace-->
         <topicName>/scan</topicName>
+        <!--updateRate>7.0</updateRate-->
         <frameName>hokuyo_link</frameName>
       </plugin>

File: nadie_description/urdf/nadie.urdf.xacro (robot description, xacro)
@@ -1,8 +1,26 @@
 <?xml version="1.0"?>
+<!--
+Copyright (c) 2018 Michael Wimble
+Permission is hereby granted, free of charge, to any person obtaining a copy
+of this software and associated documentation files (the "Software"), to deal
+in the Software without restriction, including without limitation the rights
+to use, copy, modify, merge, publish, distribute, sublicense, and/or sell
+copies of the Software, and to permit persons to whom the Software is
+furnished to do so, subject to the following conditions:
+The above copyright notice and this permission notice shall be included in all
+copies or substantial portions of the Software.
+THE SOFTWARE IS PROVIDED "AS IS", WITHOUT WARRANTY OF ANY KIND, EXPRESS OR
+IMPLIED, INCLUDING BUT NOT LIMITED TO THE WARRANTIES OF MERCHANTABILITY,
+FITNESS FOR A PARTICULAR PURPOSE AND NONINFRINGEMENT. IN NO EVENT SHALL THE
+AUTHORS OR COPYRIGHT HOLDERS BE LIABLE FOR ANY CLAIM, DAMAGES OR OTHER
+LIABILITY, WHETHER IN AN ACTION OF CONTRACT, TORT OR OTHERWISE, ARISING FROM,
+OUT OF OR IN CONNECTION WITH THE SOFTWARE OR THE USE OR OTHER DEALINGS IN THE
+SOFTWARE.
+-->
 <robot xmlns:xacro="http://ros.org/wiki/xacro" name="nadie">
   <xacro:arg name="robot_namespace" default="/nadie" />
-  <xacro:include filename="$(find nadie_control)/urdf/caster.urdf.xacro" />
-  <xacro:include filename="$(find nadie_control)/urdf/wheel.urdf.xacro" />
-  <!--xacro:include filename="$(find nadie_control)/urdf/lidar_sim.xacro" /-->
+  <xacro:include filename="$(find nadie_description)/urdf/caster.urdf.xacro" />
+  <xacro:include filename="$(find nadie_description)/urdf/wheel.urdf.xacro" />
+  <!--xacro:include filename="$(find nadie_description)/urdf/lidar_sim.xacro" /-->
   <xacro:property name="M_PI" value="3.14159"/>
   <xacro:property name="wheel_vertical_offset" value="0.03282" />
@@ -28,15 +46,4 @@
     <color rgba="0.6 0.5 0.5 1" />
   </material>
-  <!--xacro:include filename="$(find m1)/robots/m1.gazebo" /-->
-  <gazebo>
-    <plugin name="gazebo_ros_control" filename="libgazebo_ros_control.so">
-      <!-- controlPeriod defaults to parent_model_->GetWorld()->Physics()->GetMaxStepSize() -->
-      <!-- eStopTopic if specified, subscribe to this topic and capture 'data' value -->
-      <legacyModeNS>false</legacyModeNS> <!-- If using DefaultRobotHWSim, set this to "true" to fix namespace issue -->
-      <robotNamespace>$(arg robot_namespace)</robotNamespace> <!-- parent_model_->GetName() -->
-      <!--robotParam>robot_description</robotParam--> <!-- robot_description -->
-      <!--robotSimType>gazebo_ros_control/DefaultRobotHWSim</robotSimType--> <!-- gazebo_ros_control/DefaultRobotHWSim, which becomes the controller manager -->
-    </plugin>
-  </gazebo>
   <!-- Parts -->
   <link name="base_link">
@@ -103,5 +110,5 @@
       <origin xyz="0 0 0" rpy="0 0 0"/>
       <geometry>
-        <mesh filename="package://nadie_control/meshes/hokuyo.dae"/>
+        <mesh filename="package://nadie_description/meshes/hokuyo.dae"/>
       </geometry>
     </visual>
@@ -118,38 +125,4 @@
     <child link="hokuyo_link"/>
   </joint>
-  <gazebo reference="hokuyo_link">
-    <sensor type="ray" name="head_hokuyo_sensor">
-      <pose>0 0 0 0 0 0</pose>
-      <visualize>true</visualize>
-      <update_rate>7</update_rate>
-      <ray>
-        <scan>
-          <horizontal>
-            <samples>360</samples>
-            <resolution>1</resolution>
-            <min_angle>-3.14159</min_angle>
-            <max_angle>3.14159</max_angle>
-          </horizontal>
-        </scan>
-        <range>
-          <min>0.10</min>
-          <max>10.0</max>
-          <resolution>0.01</resolution>
-        </range>
-        <noise>
-          <type>gaussian</type>
-          <mean>0.0</mean>
-          <stddev>0.01</stddev>
-        </noise>
-      </ray>
-      <plugin name="gazebo_ros_head_hokuyo_controller" filename="libgazebo_ros_laser.so">
-        <alwaysOn>false</alwaysOn>
-        <!--robotNamespace></robotNamespace-->
-        <topicName>/scan</topicName>
-        <!--updateRate>7.0</updateRate-->
-        <frameName>hokuyo_link</frameName>
-      </plugin>
-    </sensor>
-  </gazebo>
   <!--link name="neato">
     <collision>

File: nadie_description/urdf/wheel.urdf.xacro (robot description, xacro)
@@ -1,3 +1,21 @@
 <?xml version="1.0"?>
+<!--
+Copyright (c) 2018 Michael Wimble
+Permission is hereby granted, free of charge, to any person obtaining a copy
+of this software and associated documentation files (the "Software"), to deal
+in the Software without restriction, including without limitation the rights
+to use, copy, modify, merge, publish, distribute, sublicense, and/or sell
+copies of the Software, and to permit persons to whom the Software is
+furnished to do so, subject to the following conditions:
+The above copyright notice and this permission notice shall be included in all
+copies or substantial portions of the Software.
+THE SOFTWARE IS PROVIDED "AS IS", WITHOUT WARRANTY OF ANY KIND, EXPRESS OR
+IMPLIED, INCLUDING BUT NOT LIMITED TO THE WARRANTIES OF MERCHANTABILITY,
+FITNESS FOR A PARTICULAR PURPOSE AND NONINFRINGEMENT. IN NO EVENT SHALL THE
+AUTHORS OR COPYRIGHT HOLDERS BE LIABLE FOR ANY CLAIM, DAMAGES OR OTHER
+LIABILITY, WHETHER IN AN ACTION OF CONTRACT, TORT OR OTHERWISE, ARISING FROM,
+OUT OF OR IN CONNECTION WITH THE SOFTWARE OR THE USE OR OTHER DEALINGS IN THE
+SOFTWARE.
+-->
 <robot xmlns:xacro="http://ros.org/wiki/xacro" name="wheel">
 	<xacro:macro name="wheel" params="wheel_prefix *joint_pose">

Commit message: Fixes to urdf

File: nadie_description/urdf/caster.urdf.xacro (robot description, xacro)
@@ -29,5 +29,5 @@
 				<origin xyz="0 0 0" rpy="${M_PI/2} 0 0" />
 				<geometry>
-			        <cylinder length="${wheel_width}" radius="${wheel_radius}" />
+			        <cylinder length="${caster_width}" radius="${caster_radius}" />
 				</geometry>
 		        <material name="wheel" />
@@ -36,5 +36,5 @@
 				<origin xyz="0 0 0" rpy="${M_PI/2} 0 0" />
 				<geometry>
-			        <cylinder length="${wheel_width}" radius="${wheel_radius}" />
+			        <cylinder length="${caster_width}" radius="${caster_radius}" />
 				</geometry>
 			</collision>

File: nadie_description/urdf/nadie.urdf.xacro (robot description, xacro)
@@ -30,20 +30,22 @@
   <!--xacro:include filename="$(find nadie_description)/urdf/lidar_sim.xacro" /-->
   <xacro:property name="M_PI" value="3.14159"/>
-  <xacro:property name="wheel_vertical_offset" value="0.03282" />
-  <xacro:property name="body_height" value="0.0508" />
-  <xacro:property name="body_length" value="0.3048" />
-  <xacro:property name="body_width" value="0.2286" />
-  <xacro:property name="fwheel_offset" value="-0.13" />
-  <xacro:property name="wheel_forward_of_center_distance" value=".0762" />
-  <xacro:property name="motor_height" value="0.0254" />
-  <xacro:property name="lidar_height" value="0.015" />
-  <xacro:property name="lidar_length" value="0.045" />
-  <xacro:property name="lidar_width" value="0.015" />
-  <xacro:property name="wheel_radius" value="0.06" />
+  <xacro:property name="wheel_distance_from_back" value="0.281" />
+  <xacro:property name="body_height" value="0.235" />
+  <xacro:property name="body_length" value="0.460" />
+  <xacro:property name="body_width" value="0.355" />
+  <xacro:property name="caster_radius" value="0.05" />
+  <xacro:property name="caster_width" value="0.030" />
+  <xacro:property name="fwheel_offset" value="${(-body_length/2)+caster_radius}" />
+  <xacro:property name="wheel_forward_of_center_distance" value="${wheel_distance_from_back-(body_length/2)}" />
+  <xacro:property name="lidar_height" value="0.05" />
+  <xacro:property name="lidar_length" value="0.125" />
+  <xacro:property name="lidar_width" value="0.1" />
+  <xacro:property name="gear_box_center_height" value="0.021" />
+  <xacro:property name="wheel_radius" value="0.1016" />
+  <xacro:property name="wheel_vertical_offset" value="${wheel_radius+gear_box_center_height}" />
   <xacro:property name="wheel_spacer" value="0.00254" />
-  <xacro:property name="wheel_width" value="0.060" />
-  <xacro:property name="body_center_height" value="${wheel_radius+(motor_height/2)+(body_height/2)}" />
-  <xacro:property name="lidar_x_offset" value="${(body_length/2)-(lidar_width/2)}" />
-  <xacro:property name="lidar_z_offset" value="${body_center_height+(body_height/2)+(lidar_height/2)+.00508}" />
+  <xacro:property name="wheel_width" value="0.040" />
+  <xacro:property name="lidar_x_offset" value="${0.105 - (body_length/2)}" />
+  <xacro:property name="lidar_z_offset" value="${body_height+(lidar_height/2)}" />
   <material name="base">
     <color rgba="0.25 0.25 0.53 1" />>
@@ -56,14 +58,14 @@
     <collision>
       <geometry>
-        <box size="${body_length+0.16} ${body_width+0.16} 0.0508"/>
+        <box size="${body_length} ${body_width} ${body_height}"/>
       </geometry>
-      <origin rpy="0 0 0" xyz="0 0 ${body_center_height}"/>
+      <origin rpy="0 0 0" xyz="0 0 ${(body_height/2)}"/>
     </collision>
     <visual>
       <geometry>
-        <box size="${body_length} ${body_width} 0.0508"/>
+        <box size="${body_length} ${body_width} ${body_height}"/>
       </geometry>
       <material name="base" />
-      <origin rpy="0 0 0" xyz="0 0 ${body_center_height}"/>
+      <origin rpy="0 0 0" xyz="0 0 ${(body_height/2)}"/>
     </visual>
     <inertial>
@@ -79,12 +81,12 @@
   <link name="base_footprint"/>
   <joint name="base_footprint_joint" type="fixed">
-    <origin xyz="0 0 ${wheel_vertical_offset - wheel_radius}" rpy="0 0 0" />
-    <parent link="base_link" />
-    <child link="base_footprint" />
+    <origin xyz="0 0 ${wheel_vertical_offset}" rpy="0 0 0" />
+    <parent link="base_footprint" />
+    <child link="base_link" />
   </joint>
   <!-- Interial link stores the robot's inertial information -->
   <link name="inertial_link">
     <inertial>
-      <mass value="46.034" />
+      <mass value="14" />
       <origin xyz="-0.00065 -0.085 0.062" />
       <inertia ixx="0.6022" ixy="-0.02364" ixz="-0.1197" iyy="1.7386" iyz="-0.001544" izz="2.0296" />
@@ -97,11 +99,14 @@
   </joint>
   <xacro:wheel wheel_prefix="front_left">
-    <origin xyz="${wheel_forward_of_center_distance} ${(body_width/2)+wheel_spacer+(wheel_width/2)} ${wheel_vertical_offset}" rpy="0 0 0" />
+    <origin xyz="${wheel_forward_of_center_distance} ${(body_width/2)+wheel_spacer+(wheel_width/2)} -${gear_box_center_height}" rpy="0 0 0" />
   </xacro:wheel>
-  <xacro:wheel wheel_prefix="front_right">
-    <origin xyz="${wheel_forward_of_center_distance} -${(body_width/2)+wheel_spacer+(wheel_width/2)} ${wheel_vertical_offset}" rpy="0 0 0" />
+ <xacro:wheel wheel_prefix="front_right">
+    <origin xyz="${wheel_forward_of_center_distance} -${(body_width/2)+wheel_spacer+(wheel_width/2)} -${gear_box_center_height}" rpy="0 0 0" />
   </xacro:wheel>
-  <xacro:caster wheel_prefix="caster">
-    <origin xyz="${fwheel_offset} 0 ${wheel_vertical_offset}" rpy="0 0 0" />
+  <xacro:caster wheel_prefix="lcaster">
+    <origin xyz="${fwheel_offset} 0.135 -${caster_radius}" rpy="0 0 0" />
+  </xacro:caster>
+  <xacro:caster wheel_prefix="rcaster">
+    <origin xyz="${fwheel_offset} -0.135 -${caster_radius}" rpy="0 0 0" />
   </xacro:caster>
   <link name="neato">
