Commit message: Adding arduino directory. More fixes for move_base

File: nadie_description/urdf/nadie.urdf.xacro (robot description, xacro)
@@ -56,5 +56,5 @@
     <collision>
       <geometry>
-        <box size="${body_length} ${body_width} 0.0508"/>
+        <box size="${body_length+0.16} ${body_width+0.16} 0.0508"/>
       </geometry>
       <origin rpy="0 0 0" xyz="0 0 ${body_center_height}"/>

Commit message: Working on nadie_rs.launch

File: nadie_description/urdf/nadie.urdf.xacro (robot description, xacro)
@@ -66,5 +66,5 @@
         <box size="${body_length} ${body_width} ${body_height}"/>
       </geometry>
-      <origin rpy="0 0 0" xyz="0 0 ${(body_height/2)}"/>
+      <origin rpy="0 0.0261799 0" xyz="0 0 ${(body_height/2)}"/>
     </collision>
     <visual>
@@ -84,5 +84,5 @@
   <link name="base_footprint"/>
   <joint name="base_footprint_joint" type="fixed">
-    <origin xyz="0 0 ${wheel_vertical_offset}" rpy="0 0 0" />
+    <origin xyz="0 0 ${wheel_vertical_offset}" rpy="0 -0.07 0" />
     <parent link="base_footprint" />
     <child link="base_link" />

Commit message: Mostly changes in tf/urdf

File: nadie_description/urdf/nadie.urdf.xacro (robot description, xacro)
@@ -144,5 +144,5 @@
   <xacro:property name="d435_length" value="0.090" />
   <xacro:property name="d435_width" value="0.025" />
-<link name="d435">
+<link name="d435_link">
     <collision>
       <geometry>
@@ -166,5 +166,5 @@
   <joint name="base_to_d435" type="fixed">
     <parent link="base_link" />
-    <child link="d435" />
+    <child link="d435_link" />
     <origin xyz="${(body_length/2)+(0.025/2)} 0 ${(-body_height/2)+0.205}" rpy="0 0 0" />
   </joint>
@@ -175,5 +175,5 @@
   <xacro:property name="t265_length" value="0.100" />
   <xacro:property name="t265_width" value="0.008" />
-  <link name="t265">
+  <link name="t265_odom_frame">
     <collision>
       <geometry>
@@ -197,5 +197,5 @@
   <joint name="base_to_t265" type="fixed">
     <parent link="base_link" />
-    <child link="t265" />
+    <child link="t265_odom_frame" />
     <origin xyz="${(body_length/2)+(0.008/2)} 0 ${(-body_height/2)+0.166}" rpy="0 0 0" />
   </joint>

Commit message: Fixes for left/right cameras

File: nadie_description/urdf/nadie.urdf.xacro (robot description, xacro)
@@ -144,5 +144,5 @@
   <xacro:property name="d435_length" value="0.090" />
   <xacro:property name="d435_width" value="0.025" />
-<link name="d435_link">
+<link name="d435_left_link">
     <collision>
       <geometry>
@@ -164,8 +164,33 @@
     </visual>
   </link>
-  <joint name="base_to_d435" type="fixed">
-    <parent link="base_link" />
-    <child link="d435_link" />
-    <origin xyz="${(body_length/2)+(0.025/2)} 0 ${(-body_height/2)+0.205}" rpy="0 0 0" />
+  <joint name="base_to_d435_left" type="fixed">
+    <parent link="base_link" />
+    <child link="d435_left_link" />
+    <origin xyz="0.245 0.055 0.180" rpy="${M_PI} 0 ${M_PI / 4}" />
+  </joint>
+<link name="d435_right_link">
+    <collision>
+      <geometry>
+        <box size="${d435_width} ${d435_length} ${d435_height}" />
+        <origin xyz="0 0 0" rpy="0 0 0" />
+      </geometry>
+    </collision>
+    <inertial>
+      <origin xyz="0 0 0" rpy="0 0 0" />
+      <mass value="1" />
+      <inertia ixx="1.0" ixy="0.0" ixz="0.0" iyy="1.0" iyz="0.0" izz="1.0" />
+    </inertial>
+    <visual>
+      <geometry>
+        <box size="${d435_width} ${d435_length} ${d435_height}" />
+      </geometry>
+      <origin xyz="0 0 0" rpy="0 0 0" />
+      <material name="d435_material" />
+    </visual>
+  </link>
+  <joint name="base_to_d435_right" type="fixed">
+    <parent link="base_link" />
+    <child link="d435_right_link" />
+    <origin xyz="0.245 -0.055 0.180" rpy="0 0 ${-M_PI / 4}" />
   </joint>
   <material name="t265_material">
@@ -198,5 +223,5 @@
     <parent link="base_link" />
     <child link="t265_odom_frame" />
-    <origin xyz="${(body_length/2)+(0.008/2)} 0 ${(-body_height/2)+0.166}" rpy="0 0 0" />
+    <origin xyz="${0.18+(0.008/2)} 0 0.15" rpy="0 0 0" />
   </joint>
 </robot>

Commit message: Adjustments to urdf after adding angle correction blocks to cameras

File: nadie_description/urdf/nadie.urdf.xacro (robot description, xacro)
@@ -167,5 +167,5 @@
     <parent link="base_link" />
     <child link="d435_left_link" />
-    <origin xyz="0.245 0.055 0.180" rpy="${M_PI} 0 ${M_PI / 4}" />
+    <origin xyz="0.30 0.042 0.180" rpy="${M_PI} 0 0.43" />
   </joint>
 <link name="d435_right_link">
@@ -192,5 +192,5 @@
     <parent link="base_link" />
     <child link="d435_right_link" />
-    <origin xyz="0.245 -0.055 0.180" rpy="0 0 ${-M_PI / 4}" />
+    <origin xyz="0.24 -0.042 0.180" rpy="0 0 -0.43" />
   </joint>
   <material name="t265_material">

Commit message: Tuning t265 parameters

File: nadie_description/urdf/nadie.urdf.xacro (robot description, xacro)
@@ -167,5 +167,5 @@
     <parent link="base_link" />
     <child link="d435_left_link" />
-    <origin xyz="0.30 0.042 0.180" rpy="${M_PI} 0 0.43" />
+    <origin xyz="0.305 0.042 0.180" rpy="${M_PI} 0 0.43" />
   </joint>
 <link name="d435_right_link">
@@ -192,5 +192,5 @@
     <parent link="base_link" />
     <child link="d435_right_link" />
-    <origin xyz="0.24 -0.042 0.180" rpy="0 0 -0.43" />
+    <origin xyz="0.305 -0.042 0.180" rpy="0 0 -0.43" />
   </joint>
   <material name="t265_material">
@@ -223,5 +223,5 @@
     <parent link="base_link" />
     <child link="t265_odom_frame" />
-    <origin xyz="${0.18+(0.008/2)} 0 0.15" rpy="0 0 0" />
+    <origin xyz="${0.24+(0.008/2)} 0 0.105" rpy="0 0 0" />
   </joint>
 </robot>

Commit message: New attempt at t265 launch

File: nadie_description/urdf/nadie.urdf.xacro (robot description, xacro)
@@ -221,6 +221,8 @@
   </link>
   <joint name="base_to_t265" type="fixed">
-    <parent link="base_link" />
-    <child link="t265_odom_frame" />
+    <!--parent link="base_link" />
+    <child link="t265_odom_frame" /-->
+    <parent link="t265_odom_frame" />
+    <child link="base_footprint" />
     <origin xyz="${0.24+(0.008/2)} 0 0.105" rpy="0 0 0" />
   </joint>

Commit message: Adding missing changes

File: nadie_description/urdf/nadie.urdf.xacro (robot description, xacro)
@@ -22,5 +22,6 @@
   <gazebo>
     <plugin name="gazebo_ros_control" filename="libgazebo_ros_control.so">
-      <legacyModeNS>true</legacyModeNS>      <!-- If using DefaultRobotHWSim, set this to "true" to fix namespace issue -->
+      <legacyModeNS>true</legacyModeNS>
+      <!-- If using DefaultRobotHWSim, set this to "true" to fix namespace issue -->
       <!--robotNamespace>$(arg robot_namespace)</robotNamespace-->
     </plugin>
@@ -200,5 +201,5 @@
   <xacro:property name="t265_length" value="0.100" />
   <xacro:property name="t265_width" value="0.008" />
-  <link name="t265_odom_frame">
+  <link name="t265_camera_link">
     <collision>
       <geometry>
@@ -221,8 +222,6 @@
   </link>
   <joint name="base_to_t265" type="fixed">
-    <!--parent link="base_link" />
-    <child link="t265_odom_frame" /-->
-    <parent link="t265_odom_frame" />
-    <child link="base_footprint" />
+    <parent link="base_link" />
+    <child link="t265_camera_link" />
     <origin xyz="${0.24+(0.008/2)} 0 0.105" rpy="0 0 0" />
   </joint>

Commit message: Frames working but camera too far out

File: nadie_description/urdf/nadie.urdf.xacro (robot description, xacro)
@@ -145,5 +145,5 @@
   <xacro:property name="d435_length" value="0.090" />
   <xacro:property name="d435_width" value="0.025" />
-<link name="d435_left_link">
+  <link name="d435_left_link">
     <collision>
       <geometry>
@@ -168,7 +168,7 @@
     <parent link="base_link" />
     <child link="d435_left_link" />
-    <origin xyz="0.305 0.042 0.180" rpy="${M_PI} 0 0.43" />
-  </joint>
-<link name="d435_right_link">
+    <origin xyz="0.305 0.042 0.180" rpy="${M_PI} 0 0.69" />
+  </joint>
+  <link name="d435_right_link">
     <collision>
       <geometry>
@@ -193,5 +193,5 @@
     <parent link="base_link" />
     <child link="d435_right_link" />
-    <origin xyz="0.305 -0.042 0.180" rpy="0 0 -0.43" />
+    <origin xyz="0.305 -0.042 0.180" rpy="0 0 -0.69" />
   </joint>
   <material name="t265_material">

Commit message: Fix new camera orientation

File: nadie_description/urdf/nadie.urdf.xacro (robot description, xacro)
@@ -168,5 +168,5 @@
     <parent link="base_link" />
     <child link="d435_left_link" />
-    <origin xyz="0.305 0.042 0.180" rpy="${M_PI} 0 0.69" />
+    <origin xyz="0.305 0.042 0.180" rpy="0 0 0.69" />
   </joint>
   <link name="d435_right_link">

Commit message: Begin of fit for new stereo camera poses

File: nadie_description/urdf/nadie.urdf.xacro (robot description, xacro)
@@ -168,5 +168,5 @@
     <parent link="base_link" />
     <child link="d435_left_link" />
-    <origin xyz="0.305 0.042 0.180" rpy="0 0 0.69" />
+    <origin xyz="0.305 0.0 0.180" rpy="0 0 0.95" />
   </joint>
   <link name="d435_right_link">
@@ -193,5 +193,5 @@
     <parent link="base_link" />
     <child link="d435_right_link" />
-    <origin xyz="0.305 -0.042 0.180" rpy="0 0 -0.69" />
+    <origin xyz="0.305 -0.0 0.180" rpy="0 0 -0.95" />
   </joint>
   <material name="t265_material">

Commit message: More changes for D435 positions

File: nadie_description/urdf/nadie.urdf.xacro (robot description, xacro)
@@ -168,5 +168,5 @@
     <parent link="base_link" />
     <child link="d435_left_link" />
-    <origin xyz="0.305 0.0 0.180" rpy="0 0 0.95" />
+    <origin xyz="0.305 0.0 0.180" rpy="0 0 0.6" />
   </joint>
   <link name="d435_right_link">
@@ -193,5 +193,5 @@
     <parent link="base_link" />
     <child link="d435_right_link" />
-    <origin xyz="0.305 -0.0 0.180" rpy="0 0 -0.95" />
+    <origin xyz="0.305 -0.0 0.180" rpy="0 0 -0.6" />
   </joint>
   <material name="t265_material">

Commit message: Changes after new physical measurements

File: nadie_description/urdf/nadie.urdf.xacro (robot description, xacro)
@@ -31,5 +31,4 @@
   <!--xacro:include filename="$(find nadie_description)/urdf/lidar_sim.xacro" /-->
   <xacro:property name="M_PI" value="3.14159"/>
-  <xacro:property name="wheel_distance_from_back" value="0.281" />
   <xacro:property name="body_height" value="0.235" />
   <xacro:property name="body_length" value="0.460" />
@@ -38,5 +37,4 @@
   <xacro:property name="caster_width" value="0.030" />
   <xacro:property name="fwheel_offset" value="${(-body_length/2)+caster_radius}" />
-  <xacro:property name="wheel_forward_of_center_distance" value="${wheel_distance_from_back-(body_length/2)}" />
   <xacro:property name="lidar_height" value="0.05" />
   <xacro:property name="lidar_length" value="0.125" />
@@ -74,5 +72,5 @@
       </geometry>
       <material name="base" />
-      <origin rpy="0 0 0" xyz="0 0 ${(body_height/2)}"/>
+      <origin rpy="0 0 0" xyz="-0.05 0 ${(body_height/2)}"/>
     </visual>
     <inertial>
@@ -85,9 +83,9 @@
   <link name="base_footprint"/>
   <joint name="base_footprint_joint" type="fixed">
-    <origin xyz="0 0 ${wheel_vertical_offset}" rpy="0 -0.07 0" />
-    <parent link="base_footprint" />
-    <child link="base_link" />
-  </joint>
-  <!-- Interial link stores the robot's inertial information -->
+    <origin xyz="0 0 -${wheel_vertical_offset}" rpy="0 -0.009599311 0" />
+    <parent link="base_link" />
+    <child link="base_footprint" />
+  </joint>
+  <!-- inetial_link stores the robot's inertial information -->
   <link name="inertial_link">
     <inertial>
@@ -103,14 +101,14 @@
   </joint>
   <xacro:wheel wheel_prefix="front_left">
-    <origin xyz="${wheel_forward_of_center_distance} ${(body_width/2)+wheel_spacer+(wheel_width/2)} -${gear_box_center_height}" rpy="0 0 0" />
+    <origin xyz="0 ${(body_width/2)+wheel_spacer+(wheel_width/2)} -${gear_box_center_height}" rpy="0 0 0" />
   </xacro:wheel>
   <xacro:wheel wheel_prefix="front_right">
-    <origin xyz="${wheel_forward_of_center_distance} -${(body_width/2)+wheel_spacer+(wheel_width/2)} -${gear_box_center_height}" rpy="0 0 0" />
+    <origin xyz="0 -${(body_width/2)+wheel_spacer+(wheel_width/2)} -${gear_box_center_height}" rpy="0 0 0" />
   </xacro:wheel>
   <xacro:caster wheel_prefix="lcaster">
-    <origin xyz="${fwheel_offset} 0.135 -${caster_radius}" rpy="0 0 0" />
+    <origin xyz="${fwheel_offset} 0.135 -${wheel_vertical_offset-caster_radius}" rpy="0 0 0" />
   </xacro:caster>
   <xacro:caster wheel_prefix="rcaster">
-    <origin xyz="${fwheel_offset} -0.135 -${caster_radius}" rpy="0 0 0" />
+    <origin xyz="${fwheel_offset} -0.135 -${wheel_vertical_offset-caster_radius}" rpy="0 0 0" />
   </xacro:caster>
   <link name="neato">
@@ -168,5 +166,5 @@
     <parent link="base_link" />
     <child link="d435_left_link" />
-    <origin xyz="0.305 0.0 0.180" rpy="0 0 0.6" />
+    <origin xyz="0.250 0.009 0.210" rpy="0 0 0.6" />
   </joint>
   <link name="d435_right_link">
@@ -193,5 +191,5 @@
     <parent link="base_link" />
     <child link="d435_right_link" />
-    <origin xyz="0.305 -0.0 0.180" rpy="0 0 -0.6" />
+    <origin xyz="0.250 0.0 0.240" rpy="0 0 -0.6" />
   </joint>
   <material name="t265_material">
@@ -224,5 +222,5 @@
     <parent link="base_link" />
     <child link="t265_camera_link" />
-    <origin xyz="${0.24+(0.008/2)} 0 0.105" rpy="0 0 0" />
+    <origin xyz="${0.180+(0.008/2)} -0.0034 0.106" rpy="0 0 0" />
   </joint>
 </robot>

Commit message: Incremental save to fix tf tree and add nonmotor launch for simulation

File: nadie_description/urdf/nadie.urdf.xacro (robot description, xacro)
@@ -45,5 +45,5 @@
   <xacro:property name="wheel_spacer" value="0.00254" />
   <xacro:property name="wheel_width" value="0.040" />
-  <xacro:property name="lidar_x_offset" value="${0.105 - (body_length/2)}" />
+  <xacro:property name="lidar_x_offset" value="-0.175" />
   <xacro:property name="lidar_z_offset" value="${body_height+(lidar_height/2)}" />
   <material name="base">

Commit message: Fixes for d435 depth image and pointcloud to laser conversion

File: nadie_description/urdf/nadie.urdf.xacro (robot description, xacro)
@@ -137,60 +137,11 @@
     <origin xyz="${lidar_x_offset} 0  ${lidar_z_offset}" rpy="0 0 0"/>
   </joint>
-  <material name="d435_material">
-    <color rgba="0.7 0.8 0.7 1" />
-  </material>
-  <xacro:property name="d435_height" value="0.025" />
-  <xacro:property name="d435_length" value="0.090" />
-  <xacro:property name="d435_width" value="0.025" />
-  <link name="d435_left_link">
-    <collision>
-      <geometry>
-        <box size="${d435_width} ${d435_length} ${d435_height}" />
-        <origin xyz="0 0 0" rpy="0 0 0" />
-      </geometry>
-    </collision>
-    <inertial>
-      <origin xyz="0 0 0" rpy="0 0 0" />
-      <mass value="1" />
-      <inertia ixx="1.0" ixy="0.0" ixz="0.0" iyy="1.0" iyz="0.0" izz="1.0" />
-    </inertial>
-    <visual>
-      <geometry>
-        <box size="${d435_width} ${d435_length} ${d435_height}" />
-      </geometry>
-      <origin xyz="0 0 0" rpy="0 0 0" />
-      <material name="d435_material" />
-    </visual>
-  </link>
-  <joint name="base_to_d435_left" type="fixed">
-    <parent link="base_link" />
-    <child link="d435_left_link" />
+  <xacro:include filename="$(find nadie_description)/urdf/_d435.urdf.xacro" />
+  <sensor_d435 parent="base_link" name="d435_left">
     <origin xyz="0.250 0.009 0.210" rpy="0 0 0.6" />
-  </joint>
-  <link name="d435_right_link">
-    <collision>
-      <geometry>
-        <box size="${d435_width} ${d435_length} ${d435_height}" />
-        <origin xyz="0 0 0" rpy="0 0 0" />
-      </geometry>
-    </collision>
-    <inertial>
-      <origin xyz="0 0 0" rpy="0 0 0" />
-      <mass value="1" />
-      <inertia ixx="1.0" ixy="0.0" ixz="0.0" iyy="1.0" iyz="0.0" izz="1.0" />
-    </inertial>
-    <visual>
-      <geometry>
-        <box size="${d435_width} ${d435_length} ${d435_height}" />
-      </geometry>
-      <origin xyz="0 0 0" rpy="0 0 0" />
-      <material name="d435_material" />
-    </visual>
-  </link>
-  <joint name="base_to_d435_right" type="fixed">
-    <parent link="base_link" />
-    <child link="d435_right_link" />
+  </sensor_d435>
+  <sensor_d435 parent="base_link" name="d435_right">
     <origin xyz="0.250 0.0 0.240" rpy="0 0 -0.6" />
-  </joint>
+  </sensor_d435>
   <material name="t265_material">
     <color rgba="0.60 0.40 0.60 1" />

Commit message: Adjusting URDF for new D435 positions

File: nadie_description/urdf/nadie.urdf.xacro (robot description, xacro)
@@ -139,8 +139,8 @@
   <xacro:include filename="$(find nadie_description)/urdf/_d435.urdf.xacro" />
   <sensor_d435 parent="base_link" name="d435_left">
-    <origin xyz="0.250 0.009 0.210" rpy="0 0 0.6" />
+    <origin xyz="0.20 0.05 0.220" rpy="0 0 0.35" />
   </sensor_d435>
   <sensor_d435 parent="base_link" name="d435_right">
-    <origin xyz="0.250 0.0 0.240" rpy="0 0 -0.6" />
+    <origin xyz="0.20 -0.07 0.220" rpy="0 0 -0.36" />
   </sensor_d435>
   <material name="t265_material">

Commit message: Attempt to improve cartographer

File: nadie_description/urdf/nadie.urdf.xacro (robot description, xacro)
@@ -74,9 +74,9 @@
       <origin rpy="0 0 0" xyz="-0.05 0 ${(body_height/2)}"/>
     </visual>
-    <inertial>
+    <!--inertial>
       <origin xyz="0 0 0" rpy="0 0 0" />
       <mass value="1" />
       <inertia ixx="1.0" ixy="0.0" ixz="0.0" iyy="1.0" iyz="0.0" izz="1.0" />
-    </inertial>
+    </inertial-->
   </link>
   <!-- Base footprint is on the ground under the robot -->

Commit message: Changes for new robot body and replacing up1d with up1f

File: nadie_description/urdf/nadie.urdf.xacro (robot description, xacro)
@@ -31,13 +31,13 @@
   <!--xacro:include filename="$(find nadie_description)/urdf/lidar_sim.xacro" /-->
   <xacro:property name="M_PI" value="3.14159"/>
-  <xacro:property name="body_height" value="0.235" />
-  <xacro:property name="body_length" value="0.460" />
-  <xacro:property name="body_width" value="0.355" />
+  <xacro:property name="body_height" value="0.305" />
+  <xacro:property name="body_length" value="0.455" />
+  <xacro:property name="body_width" value="0.315" />
   <xacro:property name="caster_radius" value="0.05" />
   <xacro:property name="caster_width" value="0.030" />
-  <xacro:property name="fwheel_offset" value="${(-body_length/2)+caster_radius}" />
+  <xacro:property name="fwheel_offset" value="-0.300" />
   <xacro:property name="lidar_height" value="0.05" />
   <xacro:property name="lidar_length" value="0.125" />
-  <xacro:property name="lidar_width" value="0.1" />
+  <xacro:property name="lidar_width" value="0.115" />
   <xacro:property name="gear_box_center_height" value="0.021" />
   <xacro:property name="wheel_radius" value="0.1016" />
@@ -45,5 +45,8 @@
   <xacro:property name="wheel_spacer" value="0.00254" />
   <xacro:property name="wheel_width" value="0.040" />
-  <xacro:property name="lidar_x_offset" value="-0.175" />
+  <xacro:property name="stereo_plate_x_offset" value="0.170" />
+  <xacro:property name="stereo_plate_z_offset" value="0.270" />
+  <xacro:property name="d435_y_offset" value="0.077" />
+  <xacro:property name="lidar_x_offset" value="-0.130" />
   <xacro:property name="lidar_z_offset" value="${body_height+(lidar_height/2)}" />
   <material name="base">
@@ -72,5 +75,5 @@
       </geometry>
       <material name="base" />
-      <origin rpy="0 0 0" xyz="-0.05 0 ${(body_height/2)}"/>
+      <origin rpy="0 0 0" xyz="${(-body_length/2)+0.125} 0 ${(body_height/2)}"/>
     </visual>
     <!--inertial>
@@ -107,8 +110,8 @@
   </xacro:wheel>
   <xacro:caster wheel_prefix="lcaster">
-    <origin xyz="${fwheel_offset} 0.135 -${wheel_vertical_offset-caster_radius}" rpy="0 0 0" />
+    <origin xyz="${fwheel_offset} 0.135 ${-caster_radius}" rpy="0 0 0" />
   </xacro:caster>
   <xacro:caster wheel_prefix="rcaster">
-    <origin xyz="${fwheel_offset} -0.135 -${wheel_vertical_offset-caster_radius}" rpy="0 0 0" />
+    <origin xyz="${fwheel_offset} -0.135 ${-caster_radius}" rpy="0 0 0" />
   </xacro:caster>
   <link name="neato">
@@ -139,8 +142,8 @@
   <xacro:include filename="$(find nadie_description)/urdf/_d435.urdf.xacro" />
   <xacro:sensor_d435 parent="base_link" name="d435_left">
-    <origin xyz="0.20 0.05 0.220" rpy="0 0 0.35" />
+    <origin xyz="${stereo_plate_x_offset} ${d435_y_offset} ${stereo_plate_z_offset}" rpy="0 0 0.35" />
   </xacro:sensor_d435>
   <xacro:sensor_d435 parent="base_link" name="d435_right">
-    <origin xyz="0.20 -0.07 0.220" rpy="0 0 -0.36" />
+    <origin xyz="${stereo_plate_x_offset} ${-d435_y_offset} ${stereo_plate_z_offset}" rpy="0 0 -0.36" />
   </xacro:sensor_d435>
   <material name="t265_material">
@@ -173,5 +176,5 @@
     <parent link="base_link" />
     <child link="t265_camera_link" />
-    <origin xyz="${0.180+(0.008/2)} -0.0034 0.106" rpy="0 0 0" />
+    <origin xyz="${stereo_plate_x_offset} 0 ${stereo_plate_z_offset-0.030}" rpy="0 0 0" />
   </joint>
 </robot>
